File: SerialServoPCB/SerialServo.kicad_pcb (KiCad board)
At the start: 2 copper layers, 40.6 x 74.9 mm, 45 parts, among them J1 Conn_01x04, J2 Conn_01x05, J3 Conn_01x05, J4 Conn_01x03, SW1 SW_Push, SW2 SW_Push, SW3 SW_Push, U1 PIC16F1847-ISO, U2 LM358A, U3 L78L05_TO92, U4 LM7805_TO220

Commit message: PCB ordered
Routing:
- net GND: track 95.1 -> 229.6 mm, vias 0 -> 1
- net +5V: track 59.4 -> 193.2 mm, vias 0 -> 3
- net +12V: track 16.3 -> 70.5 mm, vias 0 -> 2
- net TX: track 0.00 -> 51.5 mm, vias 0 -> 1
- net RX: track 0.00 -> 45.8 mm, vias 0 -> 1
- net Enc_DO: track 0.00 -> 43.1 mm
- net Batt_V: track 2.54 -> 39.9 mm, vias 0 -> 2
- net Net-(R1-Pad1): track 0.00 -> 34.0 mm, vias 0 -> 2
- net ENC_CLK: track 0.00 -> 27.0 mm, vias 0 -> 1
- net ENC_CS: track 0.00 -> 24.7 mm, vias 0 -> 1
- net GNDA: track 67.0 -> 91.2 mm, vias 0 -> 2
- net /AN4: track 5.47 -> 25.7 mm
- net Net-(C10-Pad2): track 12.9 -> 21.7 mm
- net SW1_LED1: track 39.1 -> 41.8 mm, vias 1 -> 2
- net Net-(D4-Pad1): track 15.6 -> 16.9 mm, vias 0 -> 1
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Other:
- board text added: "DMFE 2018"
- board text added: "Encoder"
- board text added: "LM358AN"
- board text added: "PIC16F1847"
- board text added: "Prog"
- board text added: "Serial Servo Rev n/c"
- board text added: "Servo"

Commit message: PCb Rev A
Parts:
- added C11: 0.1uF, Capacitor_SMD:C_0805_2012Metric_Pad1.29x1.40mm_HandSolder, F.Cu at (109.2, 120.7)
- added C12: 0.1uF, Capacitor_SMD:C_0805_2012Metric_Pad1.29x1.40mm_HandSolder, F.Cu at (109.2, 129.5)
- added C13: 0.1uF, Capacitor_SMD:C_0805_2012Metric_Pad1.29x1.40mm_HandSolder, F.Cu at (109.2, 138.4)
- added J5: Conn_01x03, Connector_Molex:Molex_KK-254_AE-6410-03A_1x03_P2.54mm_Vertical, F.Cu at (116.2, 116.2)
- added J6: Conn_01x03, Connector_Molex:Molex_KK-254_AE-6410-03A_1x03_P2.54mm_Vertical, F.Cu at (116.2, 125.1)
- added J7: Conn_01x03, Connector_Molex:Molex_KK-254_AE-6410-03A_1x03_P2.54mm_Vertical, F.Cu at (116.2, 134.0)
- added R18: 1K0, Resistor_SMD:R_0805_2012Metric_Pad1.29x1.40mm_HandSolder, F.Cu at (109.2, 118.7)
- added R19: 1K0, Resistor_SMD:R_0805_2012Metric_Pad1.29x1.40mm_HandSolder, F.Cu at (109.2, 127.6)
- added R20: 1K0, Resistor_SMD:R_0805_2012Metric_Pad1.29x1.40mm_HandSolder, F.Cu at (109.2, 136.5)
- added R21: 1K0, Resistor_SMD:R_0805_2012Metric_Pad1.29x1.40mm_HandSolder, F.Cu at (88.9, 106.7)
- added R22: 1R0, Resistor_THT:R_Axial_DIN0207_L6.3mm_D2.5mm_P10.16mm_Horizontal, F.Cu at (88.4, 85.6)
- added R23: 1R0, Resistor_THT:R_Axial_DIN0207_L6.3mm_D2.5mm_P10.16mm_Horizontal, F.Cu at (88.4, 88.1)
- C10: value 0.1uF -> 1uF
- C2, C5: footprint Capacitor_THT:CP_Radial_D4.0mm_P2.00mm -> Capacitor_THT:CP_Radial_D5.0mm_P2.00mm
- D1, D2, D3, D4: footprint LED_SMD:LED_1210_3225Metric_Pad1.22x2.70mm_HandSolder -> LED_SMD:LED_0805_2012Metric_Pad1.12x1.40mm_HandSolder
- J1: footprint Connector_PinHeader_2.54mm:PinHeader_1x04_P2.54mm_Vertical -> Connector_Molex:Molex_KK-254_AE-6410-04A_1x04_P2.54mm_Vertical
- J2: footprint Connector_PinHeader_2.54mm:PinHeader_1x05_P2.54mm_Vertical -> Connector_Molex:Molex_KK-254_AE-6410-05A_1x05_P2.54mm_Vertical
- J4: footprint Connector_PinHeader_2.54mm:PinHeader_1x03_P2.54mm_Vertical -> Connector_Molex:Molex_KK-254_AE-6410-03A_1x03_P2.54mm_Vertical
- R10: value 10K -> 47K
- U2: footprint Package_DIP:DIP-8_W7.62mm_Socket_LongPads -> Package_SO:SOIC-8_3.9x4.9mm_P1.27mm
- moved J2 36.8 mm to (116.2, 102.2), turned to 270 degrees
- moved R11 26.5 mm to (97.5, 96.5), turned to 0 degrees
- moved C1 25.8 mm to (110.5, 107.3)
- moved C3 24.7 mm to (104.1, 123.2), turned to 0 degrees
- moved R4 24.2 mm to (109.9, 99.7)
- moved R9 23.8 mm to (97.5, 94.6), turned to 0 degrees
- moved R10 22.7 mm to (97.5, 98.4)
- moved R6 22.7 mm to (88.4, 80.5), turned to 0 degrees
- moved R2 21.7 mm to (104.1, 121.3), turned to 180 degrees
- moved R5 20.4 mm to (108.6, 101.6)
- moved R8 19.8 mm to (88.4, 83.0), turned to 0 degrees
- moved C10 19.1 mm to (97.5, 100.3), turned to 0 degrees
- moved U2 18.5 mm to (103.5, 97.8)
- moved C6 16.7 mm to (88.9, 108.6)
- moved R3 16.7 mm to (104.1, 110.5), turned to 180 degrees
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Connections:
- C10 pad 2: Net-(C10-Pad2) -> GND
- C2 pad 1: GND -> Net-(C2-Pad1)
- C2 pad 2: Net-(C2-Pad2) -> GND
- C5 pad 1: GNDA -> Net-(C5-Pad1)
- C5 pad 2: Net-(C5-Pad2) -> GNDA
- D5 pad 1: Net-(C2-Pad2) -> Net-(C2-Pad1)
- D6 pad 1: Net-(C5-Pad2) -> Net-(C5-Pad1)
- R11 pad 2: Net-(C10-Pad2) -> Net-(R11-Pad2)
- R9 pad 1: Net-(C10-Pad2) -> Net-(R11-Pad2)
- RV1 pad 2: /AN4 -> Net-(R21-Pad1)
- U2 pad 2: Net-(C10-Pad2) -> Net-(R11-Pad2)
- U3 pad 3: Net-(C2-Pad2) -> Net-(C2-Pad1)
- U4 pad 1: Net-(C5-Pad2) -> Net-(C5-Pad1)
Routing:
- net +5V: track 193.2 -> 72.0 mm
- net GND: track 229.6 -> 159.8 mm, vias 1 -> 0
- net +12V: track 70.5 -> 8.30 mm, vias 2 -> 0
- net TX: track 51.5 -> 0.00 mm, vias 1 -> 0
- net RX: track 45.8 -> 0.00 mm, vias 1 -> 0
- net Batt_V: track 39.9 -> 4.75 mm, vias 2 -> 0
- net Net-(R1-Pad1): track 34.0 -> 0.00 mm, vias 2 -> 0
- net Enc_DO: track 43.1 -> 16.4 mm
- net ENC_CS: track 24.7 -> 0.00 mm, vias 1 -> 0
- net Net-(C10-Pad2): track 21.7 -> 0.00 mm
- net Net-(C5-Pad2): track 21.7 -> 0.00 mm
- net PGD: track 21.5 -> 0.00 mm
- net /AN4: track 25.7 -> 4.75 mm
- net PGC: track 15.7 -> 0.00 mm
- net Net-(C5-Pad1): track 0.00 -> 15.6 mm
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Other:
- board size 40.6 x 74.9 mm -> 33.7 x 74.9 mm
- board text removed: "DMFE 2018"
- board text removed: "Encoder"
- board text removed: "LM358AN"
- board text removed: "PIC16F1847"
- board text removed: "Prog"
- board text removed: "Serial Servo Rev n/c"
- board text removed: "Servo"

Commit message: PCB Rev A work
Parts:
- removed R23: 1R0, Resistor_THT:R_Axial_DIN0207_L6.3mm_D2.5mm_P10.16mm_Horizontal
- removed U3: L78L05_TO92, Package_TO_SOT_THT:TO-92L_Wide
- removed U4: LM7805_TO220, Package_TO_SOT_SMD:TO-263-3_TabPin2
- added C14: 0.1uF, Capacitor_SMD:C_0805_2012Metric_Pad1.29x1.40mm_HandSolder, F.Cu at (104.8, 121.3)
- added J8: Conn_01x02, Connector_PinHeader_2.54mm:PinHeader_1x02_P2.54mm_Vertical, F.Cu at (97.2, 89.5)
- added VR1: L78L05_TO92, Package_TO_SOT_THT:TO-92L_Wide, F.Cu at (99.7, 101.0)
- added VR2: LM7805_TO220, Package_TO_SOT_SMD:TO-263-3_TabPin2, F.Cu at (113.7, 88.3)
- added VR3: LD1085, Package_TO_SOT_SMD:TO-263-3_TabPin2, B.Cu at (113.7, 88.3)
- D1, D2, D3, D4, SW1, SW2, SW3: moved to B.Cu
- R22: value 1R0 -> 120R; footprint Resistor_THT:R_Axial_DIN0207_L6.3mm_D2.5mm_P10.16mm_Horizontal -> Resistor_SMD:R_0805_2012Metric_Pad1.29x1.40mm_HandSolder; moved to B.Cu
- R6: footprint Resistor_THT:R_Axial_DIN0207_L6.3mm_D2.5mm_P10.16mm_Horizontal -> Resistor_SMD:R_2512_6332Metric_Pad1.49x3.40mm_HandSolder; moved to B.Cu
- R8: value 1R0 -> RRR; footprint Resistor_THT:R_Axial_DIN0207_L6.3mm_D2.5mm_P10.16mm_Horizontal -> Resistor_SMD:R_0805_2012Metric_Pad1.29x1.40mm_HandSolder; moved to B.Cu
- U1: footprint Package_DIP:DIP-18_W7.62mm_Socket_LongPads -> Package_SO:SOIC-18W_7.5x11.6mm_P1.27mm
- moved R8 31.4 mm to (114.9, 99.7), turned to 180 degrees
- moved R22 29.3 mm to (114.9, 97.8)
- moved C2 28.9 mm to (94.6, 96.5)
- moved C4 25.5 mm to (100.0, 103.5)
- moved J5 22.1 mm to (102.2, 133.3)
- moved J4 21.6 mm to (116.2, 110.5)
- moved C9 19.9 mm to (117.5, 103.5)
- moved U1 18.2 mm to (96.5, 121.3)
- moved J2 17.1 mm to (116.2, 119.4)
- moved C11 16.8 mm to (95.9, 130.8)
- moved R18 16.8 mm to (95.9, 128.9)
- moved C6 16.7 mm to (104.8, 113.7), turned to 0 degrees
- moved R21 16.7 mm to (104.8, 111.8), turned to 180 degrees
- moved D5 14.6 mm to (97.8, 82.5)
- moved J1 14.6 mm to (90.2, 82.5)
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Connections:
- R22 pad 1: GND -> Net-(C8-Pad1)
- R22 pad 2: GNDA -> Net-(R22-Pad2)
- R8 pad 1: GND -> Net-(R22-Pad2)
Routing:
- net GND: track 159.8 -> 48.7 mm
- net SW3_LED3: track 63.0 -> 5.85 mm, vias 2 -> 0
- net GNDA: track 80.7 -> 30.4 mm
- net SW2_LED2: track 54.3 -> 5.85 mm, vias 2 -> 0
- net SW1_LED1: track 49.3 -> 5.85 mm, vias 2 -> 0
- net +5V: track 72.0 -> 31.1 mm, vias 3 -> 0
- net ENC_CLK: track 23.1 -> 0.00 mm
- net Enc_DO: track 16.4 -> 0.00 mm
- net PGD: track 0.00 -> 15.8 mm, vias 0 -> 1
- net Net-(C8-Pad1): track 27.2 -> 13.5 mm
- net PGC: track 0.00 -> 13.5 mm, vias 0 -> 1
- net Net-(C5-Pad1): track 15.6 -> 27.9 mm
- net Net-(R21-Pad1): track 11.8 -> 0.00 mm
- net /AN4: track 4.75 -> 16.0 mm, vias 0 -> 2
- net Net-(C2-Pad1): track 13.7 -> 4.45 mm
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Other:
- board size 33.7 x 74.9 mm -> 33.7 x 61.6 mm

Commit message: more lines
Parts:
- moved D5 8.89 mm to (97.8, 91.4), turned to 0 degrees
- moved D6 3.17 mm to (97.8, 82.5)
- moved R6 2.62 mm to (97.8, 82.5)
- moved J8 2.01 mm to (97.8, 87.6)
- turned D1 to 180 degrees
- turned D2 to 180 degrees
- turned D3 to 180 degrees
Routing:
- net GND: track 48.7 -> 143.9 mm
- net Net-(C8-Pad1): track 13.5 -> 82.7 mm
- net +5V: track 31.1 -> 88.2 mm
- net TX: track 0.00 -> 46.4 mm
- net GNDA: track 30.4 -> 72.4 mm
- net RX: track 0.00 -> 41.3 mm
- net ENC_CS: track 0.00 -> 24.6 mm, vias 0 -> 1
- net Net-(J7-Pad2): track 0.00 -> 20.1 mm
- net ENC_CLK: track 0.00 -> 15.2 mm, vias 0 -> 1
- net Net-(J6-Pad2): track 0.00 -> 13.7 mm
- net ServoPWM: track 0.00 -> 13.1 mm
- net +12V: track 17.2 -> 29.9 mm
- net Net-(C2-Pad1): track 4.45 -> 9.80 mm
- net Net-(D3-Pad2): track 0.00 -> 3.87 mm, vias 0 -> 1
- net Net-(D2-Pad2): track 0.00 -> 3.87 mm, vias 0 -> 1
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
Commit message: Rev A PCB is ordered
Parts:
- added REF**: OSHW-Logo2_9.8x8mm_SilkScreen, Symbol:OSHW-Logo2_9.8x8mm_SilkScreen, B.Cu at (96.4, 110.0)
Routing:
- net GND: track 143.9 -> 213.3 mm, vias 0 -> 4
- net +5V: track 88.2 -> 154.4 mm, vias 0 -> 3
- net +12V: track 29.9 -> 73.1 mm, vias 0 -> 1
- net Net-(R21-Pad1): track 0.00 -> 34.9 mm, vias 0 -> 2
- net Net-(R1-Pad1): track 0.00 -> 30.0 mm, vias 0 -> 2
- net GNDA: track 72.4 -> 101.6 mm, vias 0 -> 1
- net Enc_DO: track 0.00 -> 28.3 mm, vias 0 -> 1
- net Net-(R2-Pad1): track 1.27 -> 29.1 mm, vias 0 -> 2
- net SW3_LED3: track 8.63 -> 35.1 mm, vias 1 -> 2
- net Net-(R7-Pad1): track 3.26 -> 28.3 mm, vias 0 -> 4
- net SW2_LED2: track 8.63 -> 32.5 mm, vias 1 -> 2
- net SW1_LED1: track 8.63 -> 24.8 mm, vias 1 -> 2
- net Net-(J5-Pad2): track 0.00 -> 10.3 mm, vias 0 -> 1
- net Net-(R4-Pad2): track 5.49 -> 8.35 mm, vias 0 -> 2
- net Net-(D4-Pad2): track 0.00 -> 1.72 mm, vias 0 -> 1
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Other:
- net class Default: via_dia 1.016 -> 0.7874; via_drill 0.635 -> 0.508
- board text added: "+12 GND TX RX"
- board text added: "DMFE 2018"
- board text added: "Encoder"
- board text added: "Mode"
- board text added: "Prog"
- board text added: "Serial Servo Rev A"
- board text added: "Servo"
- board text added: "Sys"

Commit message: PCB Rev B
Parts:
- moved C9 16.5 mm to (102.2, 97.2), turned to 0 degrees
- moved J4 3.81 mm to (116.2, 106.7)
- moved J2 2.54 mm to (116.2, 116.8)
Connections:
- J3 pad 1: +5V -> VPP
- J3 pad 2: VPP -> +5V
- J3 pad 4: PGC -> PGD
- J3 pad 5: PGD -> PGC
Routing:
- net +5V: track 154.4 -> 165.3 mm, vias 3 -> 4
- net Net-(C8-Pad1): track 84.2 -> 93.1 mm
- net VPP: track 4.61 -> 7.99 mm
- net PGD: track 16.3 -> 14.0 mm
- net /AN4: track 16.7 -> 18.8 mm
- net GNDA: track 101.6 -> 99.6 mm
- net GND: track 213.3 -> 214.9 mm, vias 4 -> 5
- net ServoPWM: track 13.1 -> 11.5 mm
- net ENC_CS: track 24.7 -> 26.2 mm
- net TX: track 46.6 -> 47.6 mm
- net Enc_DO: track 28.3 -> 27.3 mm
- net +12V: track 73.1 -> 72.3 mm
- net RX: track 41.3 -> 42.0 mm
- net Net-(R21-Pad1): track 34.9 -> 34.2 mm
- net ENC_CLK: track 15.2 -> 15.8 mm
Other:
- board text added: "+5 CS G CLK DO"
- board text added: "S + -"
- board text added: "Serial Servo Rev B"
- board text removed: "Serial Servo Rev A"
