File: SerialServoPCB/SerialServo.sch (KiCad schematic (older format))
At the start: 11 parts

Commit message: Schematic 1.0
Parts:
- added C1, C10, C3, C6, C7, C8: 0.1uF, Capacitor_SMD:C_0805_2012Metric_Pad1.15x1.50mm_HandSolder, symbol Device:C_Small
- added C5: 2.2uF, Capacitor_THT:CP_Radial_D4.0mm_P2.00mm, symbol Device:C_Small
- added C9: 100uF, Capacitor_THT:CP_Radial_D8.0mm_P5.00mm, symbol Device:CP1_Small
- added D2, D3, D4: LED, LED_SMD:LED_1206_3216Metric_Pad1.07x1.80mm_HandSolder, symbol Device:LED
- added D6: D, Diode_SMD:D_SMA_Handsoldering, symbol Device:D
- added J2, J3: Conn_01x05, Connector_PinHeader_2.54mm:PinHeader_1x05_P2.54mm_Vertical, symbol Connector_Generic:Conn_01x05
- added J4: Conn_01x03, Connector_PinHeader_2.54mm:PinHeader_1x03_P2.54mm_Vertical, symbol Connector_Generic:Conn_01x03
- added R1: 220R, Resistor_SMD:R_0805_2012Metric_Pad1.15x1.50mm_HandSolder, symbol Device:R
- added R10, R11, R5: 10K, Resistor_SMD:R_0805_2012Metric_Pad1.15x1.50mm_HandSolder, symbol Device:R
- added R14, R16, R2, R3, R7: 1K0, Resistor_SMD:R_0805_2012Metric_Pad1.15x1.50mm_HandSolder, symbol Device:R
- added R15, R17: 47K, Resistor_SMD:R_0805_2012Metric_Pad1.15x1.50mm_HandSolder, symbol Device:R
- added R4, R9: 100K, Resistor_SMD:R_0805_2012Metric_Pad1.15x1.50mm_HandSolder, symbol Device:R
- added R6, R8: 1R0, Resistor_THT:R_Axial_DIN0207_L6.3mm_D2.5mm_P10.16mm_Horizontal, symbol Device:R
- added RV1: 20K, Potentiometer_THT:Potentiometer_Bourns_3296W_Vertical, symbol Device:R_POT
- added SW2, SW3: SW_Push, Button_Switch_SMD:SW_SPST_FSMSM, symbol Switch:SW_Push
- added U2: LM358A, Package_DIP:DIP-8_W7.62mm_Socket_LongPads, symbol Amplifier_Operational:LM358
- C2: renamed from C?; value C_Small -> 2.2uF; footprint (none) -> Capacitor_THT:CP_Radial_D4.0mm_P2.00mm
- C4: renamed from C?; value C_Small -> 0.1uF; footprint (none) -> Capacitor_SMD:C_0805_2012Metric_Pad1.15x1.50mm_HandSolder
- D1: renamed from D?; footprint (none) -> LED_SMD:LED_1206_3216Metric_Pad1.07x1.80mm_HandSolder
- D5: renamed from D?; footprint (none) -> Diode_SMD:D_SMA_Handsoldering
- J1: renamed from J?; footprint (none) -> Connector_PinHeader_2.54mm:PinHeader_1x04_P2.54mm_Vertical
- R12: renamed from R?; value R -> 1K0; footprint (none) -> Resistor_SMD:R_0805_2012Metric_Pad1.15x1.50mm_HandSolder
- R13: renamed from R?; value R -> 47K; footprint (none) -> Resistor_SMD:R_0805_2012Metric_Pad1.15x1.50mm_HandSolder
- SW1: renamed from SW?; footprint (none) -> Button_Switch_SMD:SW_SPST_FSMSM
- U1: renamed from U?; footprint (none) -> Package_DIP:DIP-18_W7.62mm_Socket_LongPads
- U3: renamed from U?; footprint Package_TO_SOT_THT:TO-92_Inline -> Package_TO_SOT_THT:TO-92L_Wide
- U4: renamed from U?; footprint Package_TO_SOT_THT:TO-220-3_Vertical -> Package_TO_SOT_SMD:TO-263-3_TabPin2
Connections:
- net labels added: +12V, AN0, AN4, Batt_V, ENC_CLK, ENC_CS, Enc_DO, GNDA, PGC, PGD, RX, SW1_LED1, SW2_LED2, SW3_LED3, ServoPWM, TX, VPP
- wire segments 0 -> 179
Other:
- note added: "Encoder"
- note added: "Input voltage 6.5 to 16 volts."
- note added: "Note: Analog Ref+ = 2.048V"
- note added: "Prog"
- note added: "System LED"
- note added: "VDD\nCS*\nVSS\nCLK\nDO"
- note added: "VDD\nVPP\nVSS\nPGC\nPGD"
- moved on the sheet: U1, U3

Commit message: Started PCB
Parts:
- C1, C10, C3, C4, C6, C7, C8: footprint Capacitor_SMD:C_0805_2012Metric_Pad1.15x1.50mm_HandSolder -> Capacitor_SMD:C_0805_2012Metric_Pad1.29x1.40mm_HandSolder
- D1, D2, D3, D4: footprint LED_SMD:LED_1206_3216Metric_Pad1.07x1.80mm_HandSolder -> LED_SMD:LED_1210_3225Metric_Pad1.22x2.70mm_HandSolder
- R1, R10, R11, R12, R13, R14, R15, R16, R17, R2, R3, R4, R5, R7, R9: footprint Resistor_SMD:R_0805_2012Metric_Pad1.15x1.50mm_HandSolder -> Resistor_SMD:R_0805_2012Metric_Pad1.29x1.40mm_HandSolder
Changed lines of the file:
@@
 F 0 "D1" H 8791 1966 50  0000 C CNN
 F 1 "LED" H 8791 1875 50  0000 C CNN
-F 2 "LED_SMD:LED_1206_3216Metric_Pad1.07x1.80mm_HandSolder" H 8800 1750 50  0001 C CNN
+F 2 "LED_SMD:LED_1210_3225Metric_Pad1.22x2.70mm_HandSolder" H 8800 1750 50  0001 C CNN
 F 3 "~" H 8800 1750 50  0001 C CNN
 	1    8800 1750
@@
 F 0 "R13" V 8993 2050 50  0000 C CNN
 F 1 "47K" V 9084 2050 50  0000 C CNN
-F 2 "Resistor_SMD:R_0805_2012Metric_Pad1.15x1.50mm_HandSolder" V 9130 2050 50  0001 C CNN
+F 2 "Resistor_SMD:R_0805_2012Metric_Pad1.29x1.40mm_HandSolder" V 9130 2050 50  0001 C CNN
 F 3 "~" H 9200 2050 50  0001 C CNN
 	1    9200 2050
@@
 F 0 "R12" V 8993 1750 50  0000 C CNN
 F 1 "1K0" V 9084 1750 50  0000 C CNN
-F 2 "Resistor_SMD:R_0805_2012Metric_Pad1.15x1.50mm_HandSolder" V 9130 1750 50  0001 C CNN
+F 2 "Resistor_SMD:R_0805_2012Metric_Pad1.29x1.40mm_HandSolder" V 9130 1750 50  0001 C CNN
 F 3 "~" H 9200 1750 50  0001 C CNN
 	1    9200 1750
@@
 F 0 "C4" H 3792 1246 50  0000 L CNN
 F 1 "0.1uF" H 3792 1155 50  0000 L CNN
-F 2 "Capacitor_SMD:C_0805_2012Metric_Pad1.15x1.50mm_HandSolder" H 3700 1200 50  0001 C CNN
+F 2 "Capacitor_SMD:C_0805_2012Metric_Pad1.29x1.40mm_HandSolder" H 3700 1200 50  0001 C CNN
 F 3 "~" H 3700 1200 50  0001 C CNN
 	1    3700 1200
@@
 F 0 "C8" H 5792 1246 50  0000 L CNN
 F 1 "0.1uF" H 5792 1155 50  0000 L CNN
-F 2 "Capacitor_SMD:C_0805_2012Metric_Pad1.15x1.50mm_HandSolder" H 5700 1200 50  0001 C CNN
+F 2 "Capacitor_SMD:C_0805_2012Metric_Pad1.29x1.40mm_HandSolder" H 5700 1200 50  0001 C CNN
 F 3 "~" H 5700 1200 50  0001 C CNN
 	1    5700 1200
@@
 F 0 "R1" V 1243 3800 50  0000 C CNN
 F 1 "220R" V 1334 3800 50  0000 C CNN
-F 2 "Resistor_SMD:R_0805_2012Metric_Pad1.15x1.50mm_HandSolder" V 1380 3800 50  0001 C CNN
+F 2 "Resistor_SMD:R_0805_2012Metric_Pad1.29x1.40mm_HandSolder" V 1380 3800 50  0001 C CNN
 F 3 "~" H 1450 3800 50  0001 C CNN
 	1    1450 3800
@@
 F 0 "D2" H 8791 2716 50  0000 C CNN
 F 1 "LED" H 8791 2625 50  0000 C CNN
-F 2 "LED_SMD:LED_1206_3216Metric_Pad1.07x1.80mm_HandSolder" H 8800 2500 50  0001 C CNN
+F 2 "LED_SMD:LED_1210_3225Metric_Pad1.22x2.70mm_HandSolder" H 8800 2500 50  0001 C CNN
 F 3 "~" H 8800 2500 50  0001 C CNN
 	1    8800 2500
@@
 F 0 "R15" V 8993 2800 50  0000 C CNN
 F 1 "47K" V 9084 2800 50  0000 C CNN
-F 2 "Resistor_SMD:R_0805_2012Metric_Pad1.15x1.50mm_HandSolder" V 9130 2800 50  0001 C CNN
+F 2 "Resistor_SMD:R_0805_2012Metric_Pad1.29x1.40mm_HandSolder" V 9130 2800 50  0001 C CNN
 F 3 "~" H 9200 2800 50  0001 C CNN
 	1    9200 2800
@@
 F 0 "R14" V 8993 2500 50  0000 C CNN
 F 1 "1K0" V 9084 2500 50  0000 C CNN
-F 2 "Resistor_SMD:R_0805_2012Metric_Pad1.15x1.50mm_HandSolder" V 9130 2500 50  0001 C CNN
+F 2 "Resistor_SMD:R_0805_2012Metric_Pad1.29x1.40mm_HandSolder" V 9130 2500 50  0001 C CNN
 F 3 "~" H 9200 2500 50  0001 C CNN
 	1    9200 2500
@@
 F 0 "D3" H 8791 3466 50  0000 C CNN
 F 1 "LED" H 8791 3375 50  0000 C CNN
-F 2 "LED_SMD:LED_1206_3216Metric_Pad1.07x1.80mm_HandSolder" H 8800 3250 50  0001 C CNN
+F 2 "LED_SMD:LED_1210_3225Metric_Pad1.22x2.70mm_HandSolder" H 8800 3250 50  0001 C CNN
 F 3 "~" H 8800 3250 50  0001 C CNN
 	1    8800 3250
@@
 F 0 "R17" V 8993 3550 50  0000 C CNN
 F 1 "47K" V 9084 3550 50  0000 C CNN
-F 2 "Resistor_SMD:R_0805_2012Metric_Pad1.15x1.50mm_HandSolder" V 9130 3550 50  0001 C CNN
+F 2 "Resistor_SMD:R_0805_2012Metric_Pad1.29x1.40mm_HandSolder" V 9130 3550 50  0001 C CNN
 F 3 "~" H 9200 3550 50  0001 C CNN
 	1    9200 3550
@@
 F 0 "R16" V 8993 3250 50  0000 C CNN
 F 1 "1K0" V 9084 3250 50  0000 C CNN
-F 2 "Resistor_SMD:R_0805_2012Metric_Pad1.15x1.50mm_HandSolder" V 9130 3250 50  0001 C CNN
+F 2 "Resistor_SMD:R_0805_2012Metric_Pad1.29x1.40mm_HandSolder" V 9130 3250 50  0001 C CNN
 F 3 "~" H 9200 3250 50  0001 C CNN
 	1    9200 3250
@@
 F 0 "C10" H 6492 3546 50  0000 L CNN
 F 1 "0.1uF" H 6492 3455 50  0000 L CNN
-F 2 "Capacitor_SMD:C_0805_2012Metric_Pad1.15x1.50mm_HandSolder" H 6400 3500 50  0001 C CNN
+F 2 "Capacitor_SMD:C_0805_2012Metric_Pad1.29x1.40mm_HandSolder" H 6400 3500 50  0001 C CNN
 F 3 "~" H 6400 3500 50  0001 C CNN
 	1    6400 3500
@@
 F 0 "R10" V 6443 3300 50  0000 C CNN
 F 1 "10K" V 6534 3300 50  0000 C CNN
-F 2 "Resistor_SMD:R_0805_2012Metric_Pad1.15x1.50mm_HandSolder" V 6580 3300 50  0001 C CNN
+F 2 "Resistor_SMD:R_0805_2012Metric_Pad1.29x1.40mm_HandSolder" V 6580 3300 50  0001 C CNN
 F 3 "~" H 6650 3300 50  0001 C CNN
 	1    6650 3300
@@
 F 0 "R11" V 6443 4100 50  0000 C CNN
 F 1 "10K" V 6534 4100 50  0000 C CNN
-F 2 "Resistor_SMD:R_0805_2012Metric_Pad1.15x1.50mm_HandSolder" V 6580 4100 50  0001 C CNN
+F 2 "Resistor_SMD:R_0805_2012Metric_Pad1.29x1.40mm_HandSolder" V 6580 4100 50  0001 C CNN
 F 3 "~" H 6650 4100 50  0001 C CNN
 	1    6650 4100
@@
 F 0 "R9" V 5443 4100 50  0000 C CNN
 F 1 "100K" V 5534 4100 50  0000 C CNN
-F 2 "Resistor_SMD:R_0805_2012Metric_Pad1.15x1.50mm_HandSolder" V 5580 4100 50  0001 C CNN
+F 2 "Resistor_SMD:R_0805_2012Metric_Pad1.29x1.40mm_HandSolder" V 5580 4100 50  0001 C CNN
 F 3 "~" H 5650 4100 50  0001 C CNN
 	1    5650 4100
@@
 F 0 "R7" V 5093 3500 50  0000 C CNN
 F 1 "1K0" V 5184 3500 50  0000 C CNN
-F 2 "Resistor_SMD:R_0805_2012Metric_Pad1.15x1.50mm_HandSolder" V 5230 3500 50  0001 C CNN
+F 2 "Resistor_SMD:R_0805_2012Metric_Pad1.29x1.40mm_HandSolder" V 5230 3500 50  0001 C CNN
 F 3 "~" H 5300 3500 50  0001 C CNN
 	1    5300 3500
@@
 F 0 "C7" H 5192 3746 50  0000 L CNN
 F 1 "0.1uF" H 5192 3655 50  0000 L CNN
-F 2 "Capacitor_SMD:C_0805_2012Metric_Pad1.15x1.50mm_HandSolder" H 5100 3700 50  0001 C CNN
+F 2 "Capacitor_SMD:C_0805_2012Metric_Pad1.29x1.40mm_HandSolder" H 5100 3700 50  0001 C CNN
 F 3 "~" H 5100 3700 50  0001 C CNN
 	1    5100 3700
@@
 F 0 "C1" H 2192 5296 50  0000 L CNN
 F 1 "0.1uF" H 2192 5205 50  0000 L CNN
-F 2 "Capacitor_SMD:C_0805_2012Metric_Pad1.15x1.50mm_HandSolder" H 2100 5250 50  0001 C CNN
+F 2 "Capacitor_SMD:C_0805_2012Metric_Pad1.29x1.40mm_HandSolder" H 2100 5250 50  0001 C CNN
 F 3 "~" H 2100 5250 50  0001 C CNN
 	1    2100 5250
@@
 F 0 "D4" H 4191 5216 50  0000 C CNN
 F 1 "LED" H 4191 5125 50  0000 C CNN
-F 2 "LED_SMD:LED_1206_3216Metric_Pad1.07x1.80mm_HandSolder" H 4200 5000 50  0001 C CNN
+F 2 "LED_SMD:LED_1210_3225Metric_Pad1.22x2.70mm_HandSolder" H 4200 5000 50  0001 C CNN
 F 3 "~" H 4200 5000 50  0001 C CNN
 	1    4200 5000
@@
 F 0 "R3" V 3593 5000 50  0000 C CNN
 F 1 "1K0" V 3684 5000 50  0000 C CNN
-F 2 "Resistor_SMD:R_0805_2012Metric_Pad1.15x1.50mm_HandSolder" V 3730 5000 50  0001 C CNN
+F 2 "Resistor_SMD:R_0805_2012Metric_Pad1.29x1.40mm_HandSolder" V 3730 5000 50  0001 C CNN
 F 3 "~" H 3800 5000 50  0001 C CNN
 	1    3800 5000
@@
 F 0 "C6" H 4992 5146 50  0000 L CNN
 F 1 "0.1uF" H 4992 5055 50  0000 L CNN
-F 2 "Capacitor_SMD:C_0805_2012Metric_Pad1.15x1.50mm_HandSolder" H 4900 5100 50  0001 C CNN
+F 2 "Capacitor_SMD:C_0805_2012Metric_Pad1.29x1.40mm_HandSolder" H 4900 5100 50  0001 C CNN
 F 3 "~" H 4900 5100 50  0001 C CNN
 	1    4900 5100
@@
 F 0 "C3" H 3092 6646 50  0000 L CNN
 F 1 "0.1uF" H 3092 6555 50  0000 L CNN
-F 2 "Capacitor_SMD:C_0805_2012Metric_Pad1.15x1.50mm_HandSolder" H 3000 6600 50  0001 C CNN
+F 2 "Capacitor_SMD:C_0805_2012Metric_Pad1.29x1.40mm_HandSolder" H 3000 6600 50  0001 C CNN
 F 3 "~" H 3000 6600 50  0001 C CNN
 	1    3000 6600
@@
 F 0 "R2" V 2993 6400 50  0000 C CNN
 F 1 "1K0" V 3084 6400 50  0000 C CNN
-F 2 "Resistor_SMD:R_0805_2012Metric_Pad1.15x1.50mm_HandSolder" V 3130 6400 50  0001 C CNN
+F 2 "Resistor_SMD:R_0805_2012Metric_Pad1.29x1.40mm_HandSolder" V 3130 6400 50  0001 C CNN
 F 3 "~" H 3200 6400 50  0001 C CNN
 	1    3200 6400
@@
 F 0 "R4" V 4543 6300 50  0000 C CNN
 F 1 "100K" V 4634 6300 50  0000 C CNN
-F 2 "Resistor_SMD:R_0805_2012Metric_Pad1.15x1.50mm_HandSolder" V 4680 6300 50  0001 C CNN
+F 2 "Resistor_SMD:R_0805_2012Metric_Pad1.29x1.40mm_HandSolder" V 4680 6300 50  0001 C CNN
 F 3 "~" H 4750 6300 50  0001 C CNN
 	1    4750 6300
@@
 F 0 "R5" V 4543 6600 50  0000 C CNN
 F 1 "10K" V 4634 6600 50  0000 C CNN
-F 2 "Resistor_SMD:R_0805_2012Metric_Pad1.15x1.50mm_HandSolder" V 4680 6600 50  0001 C CNN
+F 2 "Resistor_SMD:R_0805_2012Metric_Pad1.29x1.40mm_HandSolder" V 4680 6600 50  0001 C CNN
 F 3 "~" H 4750 6600 50  0001 C CNN
 	1    4750 6600

Commit message: PCb Rev A
Parts:
- removed C2, C5: 2.2uF, Capacitor_THT:CP_Radial_D4.0mm_P2.00mm, symbol Device:C_Small
- added C11, C12, C13: 0.1uF, Capacitor_SMD:C_0805_2012Metric_Pad1.29x1.40mm_HandSolder, symbol Device:C_Small
- added C2, C5: 2.2uF, Capacitor_THT:CP_Radial_D5.0mm_P2.00mm, symbol Device:CP1_Small
- added J5, J6, J7: Conn_01x03, Connector_Molex:Molex_KK-254_AE-6410-03A_1x03_P2.54mm_Vertical, symbol Connector_Generic:Conn_01x03
- added R18, R19, R20, R21: 1K0, Resistor_SMD:R_0805_2012Metric_Pad1.29x1.40mm_HandSolder, symbol Device:R
- added R22, R23: 1R0, Resistor_THT:R_Axial_DIN0207_L6.3mm_D2.5mm_P10.16mm_Horizontal, symbol Device:R
- added unit 3 of U2
- C10: value 0.1uF -> 1uF
- D1, D2, D3, D4: footprint LED_SMD:LED_1210_3225Metric_Pad1.22x2.70mm_HandSolder -> LED_SMD:LED_0805_2012Metric_Pad1.12x1.40mm_HandSolder
- J1: footprint Connector_PinHeader_2.54mm:PinHeader_1x04_P2.54mm_Vertical -> Connector_Molex:Molex_KK-254_AE-6410-04A_1x04_P2.54mm_Vertical
- J2: footprint Connector_PinHeader_2.54mm:PinHeader_1x05_P2.54mm_Vertical -> Connector_Molex:Molex_KK-254_AE-6410-05A_1x05_P2.54mm_Vertical
- J4: footprint Connector_PinHeader_2.54mm:PinHeader_1x03_P2.54mm_Vertical -> Connector_Molex:Molex_KK-254_AE-6410-03A_1x03_P2.54mm_Vertical
- R10: value 10K -> 47K
- U2: footprint Package_DIP:DIP-8_W7.62mm_Socket_LongPads -> Package_SO:SOIC-8_3.9x4.9mm_P1.27mm
Connections:
- wire segments 179 -> 220

Commit message: PCB Rev A work
Parts:
- removed R23: 1R0, Resistor_THT:R_Axial_DIN0207_L6.3mm_D2.5mm_P10.16mm_Horizontal, symbol Device:R
- added C14: 0.1uF, Capacitor_SMD:C_0805_2012Metric_Pad1.29x1.40mm_HandSolder, symbol Device:C_Small
- added J8: Conn_01x02, Connector_PinHeader_2.54mm:PinHeader_1x02_P2.54mm_Vertical, symbol Connector_Generic:Conn_01x02
- added VR3: LD1085, Package_TO_SOT_SMD:TO-263-3_TabPin2, symbol Regulator_Linear:AZ1117-ADJ
- R22: value 1R0 -> 120R; footprint Resistor_THT:R_Axial_DIN0207_L6.3mm_D2.5mm_P10.16mm_Horizontal -> Resistor_SMD:R_0805_2012Metric_Pad1.29x1.40mm_HandSolder
- R6: footprint Resistor_THT:R_Axial_DIN0207_L6.3mm_D2.5mm_P10.16mm_Horizontal -> Resistor_SMD:R_2512_6332Metric_Pad1.49x3.40mm_HandSolder
- R8: value 1R0 -> RRR; footprint Resistor_THT:R_Axial_DIN0207_L6.3mm_D2.5mm_P10.16mm_Horizontal -> Resistor_SMD:R_0805_2012Metric_Pad1.29x1.40mm_HandSolder
- U1: footprint Package_DIP:DIP-18_W7.62mm_Socket_LongPads -> Package_SO:SOIC-18W_7.5x11.6mm_P1.27mm
- renumbered U3 to VR1, U4 to VR2
Connections:
- wire segments 220 -> 224
Other:
- note added: "Optional 3A Adj. Reg."
- note added: "V-Reg bypass"

Commit message: PCB Rev B
Parts:
- R6: value 1R0 -> 0R200 1W
Other:
- note added: "D1 blinks Mode"
- note added: "LED and Button\nor\nSwitch Input\nor\nAnalog Input\nor\nDigital Output"
- note added: "Note: Analog Ref+ = 5.0V"
- note added: "Optional"
- note added: "Optional Options"
- note added: "Power and TTL Serial"
- note added: "R1 220R\nR2,R3,R7,R12,R14,\nR16,R18,R19,R20,R21 1K0\nR4,R9 100K\nR5,R11 10K\nR6 0R20\nR8 ?K?? Adj Volts\nR10 47K\nR13 removed\nR22 120R"
- note added: "Rev. B 6/19/2018 Fixed J3 pinout, Fixed spacing of J4 to J2 to J7."
- note added: "U1 PIC16F1847\nU2 LM358A\n"
- note added: "VDD\nVPP\nVSS\nPGD\nPGC"
- note removed: "Note: Analog Ref+ = 2.048V"
- note removed: "VDD\nVPP\nVSS\nPGC\nPGD"
Changed lines of the file:
@@
 Sheet 1 1
 Title "Serial Servo"
-Date "2018-06-03"
-Rev "A"
+Date "2018-06-19"
+Rev "B"
 Comp "DMFE"
 Comment1 "TTL serial r/c servo controller"
@@
 U 1 1 5AEA83CA
 P 1200 1300
-F 0 "J1" H 1120 1617 50  0000 C CNN
-F 1 "Conn_01x04" H 1120 1526 50  0000 C CNN
+F 0 "J1" H 1300 1500 50  0000 C CNN
+F 1 "Conn_01x04" H 1120 1526 50  0001 C CNN
 F 2 "Connector_Molex:Molex_KK-254_AE-6410-04A_1x04_P2.54mm_Vertical" H 1200 1300 50  0001 C CNN
 F 3 "~" H 1200 1300 50  0001 C CNN
@@
 U 1 1 5AECF704
 P 5300 2550
-F 0 "R6" H 5350 2400 50  0000 L CNN
-F 1 "1R0" V 5300 2500 50  0000 L CNN
+F 0 "R6" H 5400 2500 50  0000 L CNN
+F 1 "0R200 1W" H 5400 2650 50  0000 L CNN
 F 2 "Resistor_SMD:R_2512_6332Metric_Pad1.49x3.40mm_HandSolder" V 5230 2550 50  0001 C CNN
 F 3 "~" H 5300 2550 50  0001 C CNN
@@
 P 6800 1900
 F 0 "J4" H 6880 1942 50  0000 L CNN
-F 1 "Conn_01x03" H 6880 1851 50  0000 L CNN
+F 1 "Conn_01x03" H 6880 1851 50  0001 L CNN
 F 2 "Connector_Molex:Molex_KK-254_AE-6410-03A_1x03_P2.54mm_Vertical" H 6800 1900 50  0001 C CNN
 F 3 "~" H 6800 1900 50  0001 C CNN
@@
 U 1 1 5AED22A3
 P 1450 3800
-F 0 "R1" V 1243 3800 50  0000 C CNN
-F 1 "220R" V 1334 3800 50  0000 C CNN
+F 0 "R1" V 1350 3750 50  0000 C CNN
+F 1 "220R" V 1450 3800 50  0000 C CNN
 F 2 "Resistor_SMD:R_0805_2012Metric_Pad1.29x1.40mm_HandSolder" V 1380 3800 50  0001 C CNN
 F 3 "~" H 1450 3800 50  0001 C CNN
@@
 Prog
 Text Notes 1750 6650 2    62   ~ 0
-VDD\nVPP\nVSS\nPGC\nPGD
+VDD\nVPP\nVSS\nPGD\nPGC
 Text GLabel 2000 4200 0    50   Input ~ 0
 PGD
-Text GLabel 1100 6600 0    50   Input ~ 0
+Text GLabel 1100 6500 0    50   Input ~ 0
 PGD
 Text GLabel 2000 4100 0    50   Input ~ 0
@@
 Text GLabel 4400 4000 2    50   Input ~ 0
 VPP
-Text GLabel 1100 6500 0    50   Input ~ 0
+Text GLabel 1100 6600 0    50   Input ~ 0
 PGC
-Text GLabel 1100 6300 0    50   Input ~ 0
+Text GLabel 1200 6200 0    50   Input ~ 0
 VPP
 $Comp
 L power:+5V #PWR02
 U 1 1 5AEDCBB7
-P 1200 6150
-F 0 "#PWR02" H 1200 6000 50  0001 C CNN
-F 1 "+5V" H 1215 6323 50  0000 C CNN
-F 2 "" H 1200 6150 50  0001 C CNN
-F 3 "" H 1200 6150 50  0001 C CNN
-	1    1200 6150
+P 900 6250
+F 0 "#PWR02" H 900 6100 50  0001 C CNN
+F 1 "+5V" H 915 6423 50  0000 C CNN
+F 2 "" H 900 6250 50  0001 C CNN
+F 3 "" H 900 6250 50  0001 C CNN
+	1    900  6250
 	1    0    0    -1
 $EndComp
@@
 Wire Wire Line
 	700  6400 700  6500
-Wire Wire Line
-	1100 6300 1250 6300
-Wire Wire Line
-	1200 6150 1200 6200
 Wire Wire Line
 	1200 6200 1250 6200
@@
 	-1   0    0    -1
 $EndComp
-Text Notes 1100 5750 0    50   ~ 0
+Text Notes 900  5850 0    100  ~ 0
 Encoder
 Text Notes 850  5650 0    62   ~ 0
@@
 U 1 1 5AF79064
 P 3800 5000
-F 0 "R3" V 3593 5000 50  0000 C CNN
-F 1 "1K0" V 3684 5000 50  0000 C CNN
+F 0 "R3" V 3900 4950 50  0000 C CNN
+F 1 "1K0" V 3800 5000 50  0000 C CNN
 F 2 "Resistor_SMD:R_0805_2012Metric_Pad1.29x1.40mm_HandSolder" V 3730 5000 50  0001 C CNN
 F 3 "~" H 3800 5000 50  0001 C CNN
@@
 U 1 1 5AFEFAFB
 P 3200 6400
-F 0 "R2" V 2993 6400 50  0000 C CNN
-F 1 "1K0" V 3084 6400 50  0000 C CNN
+F 0 "R2" V 3100 6350 50  0000 C CNN
+F 1 "1K0" V 3200 6400 50  0000 C CNN
 F 2 "Resistor_SMD:R_0805_2012Metric_Pad1.29x1.40mm_HandSolder" V 3130 6400 50  0001 C CNN
 F 3 "~" H 3200 6400 50  0001 C CNN
@@
 U 1 1 5B01A70C
 P 4750 6300
-F 0 "R4" V 4543 6300 50  0000 C CNN
-F 1 "100K" V 4634 6300 50  0000 C CNN
+F 0 "R4" V 4650 6250 50  0000 C CNN
+F 1 "100K" V 4750 6300 50  0000 C CNN
 F 2 "Resistor_SMD:R_0805_2012Metric_Pad1.29x1.40mm_HandSolder" V 4680 6300 50  0001 C CNN
 F 3 "~" H 4750 6300 50  0001 C CNN
@@
 U 1 1 5B02A185
 P 4750 6600
-F 0 "R5" V 4543 6600 50  0000 C CNN
-F 1 "10K" V 4634 6600 50  0000 C CNN
+F 0 "R5" V 4650 6550 50  0000 C CNN
+F 1 "10K" V 4750 6600 50  0000 C CNN
 F 2 "Resistor_SMD:R_0805_2012Metric_Pad1.29x1.40mm_HandSolder" V 4680 6600 50  0001 C CNN
 F 3 "~" H 4750 6600 50  0001 C CNN
@@
 	3450 6400 3600 6400
 Text Notes 6250 5250 0    50   ~ 0
-Note: Analog Ref+ = 2.048V
+Note: Analog Ref+ = 5.0V
 Text Notes 6250 5400 0    50   ~ 0
 Input voltage 6.5 to 16 volts.
@@
 U 1 1 5B1AA0CA
 P 4950 4950
-F 0 "R21" V 4743 4950 50  0000 C CNN
-F 1 "1K0" V 4834 4950 50  0000 C CNN
+F 0 "R21" V 4850 4950 50  0000 C CNN
+F 1 "1K0" V 4950 4950 50  0000 C CNN
 F 2 "Resistor_SMD:R_0805_2012Metric_Pad1.29x1.40mm_HandSolder" V 4880 4950 50  0001 C CNN
 F 3 "~" H 4950 4950 50  0001 C CNN
@@
 P 9650 1950
 F 0 "J5" H 9730 1992 50  0000 L CNN
-F 1 "Conn_01x03" H 9730 1901 50  0000 L CNN
+F 1 "Conn_01x03" H 9730 1901 50  0001 L CNN
 F 2 "Connector_Molex:Molex_KK-254_AE-6410-03A_1x03_P2.54mm_Vertical" H 9650 1950 50  0001 C CNN
 F 3 "~" H 9650 1950 50  0001 C CNN
@@
 P 9650 3100
 F 0 "J6" H 9730 3142 50  0000 L CNN
-F 1 "Conn_01x03" H 9730 3051 50  0000 L CNN
+F 1 "Conn_01x03" H 9730 3051 50  0001 L CNN
 F 2 "Connector_Molex:Molex_KK-254_AE-6410-03A_1x03_P2.54mm_Vertical" H 9650 3100 50  0001 C CNN
 F 3 "~" H 9650 3100 50  0001 C CNN
@@
 P 9650 4250
 F 0 "J7" H 9730 4292 50  0000 L CNN
-F 1 "Conn_01x03" H 9730 4201 50  0000 L CNN
+F 1 "Conn_01x03" H 9730 4201 50  0001 L CNN
 F 2 "Connector_Molex:Molex_KK-254_AE-6410-03A_1x03_P2.54mm_Vertical" H 9650 4250 50  0001 C CNN
 F 3 "~" H 9650 4250 50  0001 C CNN
@@
 	3400 2850 3200 2850
 Connection ~ 3200 2850
+Wire Wire Line
+	900  6300 900  6250
+Wire Wire Line
+	900  6300 1250 6300
+Text Notes 7850 5750 0    50   ~ 0
+R1                                220R\nR2,R3,R7,R12,R14,\nR16,R18,R19,R20,R21             1K0\nR4,R9                            100K\nR5,R11                            10K\nR6                               0R20\nR8                      ?K??  Adj Volts\nR10                              47K\nR13         removed\nR22                              120R
+Text Notes 7850 6050 0    50   ~ 0
+U1  PIC16F1847\nU2  LM358A\n
+Text Notes 7650 650  0    50   ~ 0
+Rev. B 6/19/2018  Fixed J3 pinout, Fixed spacing of J4 to J2 to J7.
+Text Notes 6250 5650 0    50   ~ 0
+D1 blinks Mode
+Wire Notes Line
+	10300 1150 10300 4750
+Wire Notes Line
+	10300 4750 7350 4750
+Wire Notes Line
+	7350 4750 7350 1150
+Wire Notes Line
+	7350 1150 10300 1150
+Wire Notes Line
+	4700 4250 5650 4250
+Wire Notes Line
+	5650 4250 5650 5600
+Wire Notes Line
+	5650 5600 4700 5600
+Wire Notes Line
+	4700 5600 4700 4250
+Text Notes 5050 4350 0    50   ~ 0
+Optional
+Text Notes 7400 1300 0    50   ~ 0
+Optional Options
+Text Notes 800  1800 0    100  ~ 0
+Power and TTL Serial
+Text Notes 7400 2650 0    50   ~ 0
+LED and Button\nor\nSwitch Input\nor\nAnalog Input\nor\nDigital Output
 $EndSCHEMATC

Commit message: little things
Other:
- note added: "VPP\nVDD\nVSS\nPGD\nPGC"
- note removed: "VDD\nVPP\nVSS\nPGD\nPGC"
Changed lines of the file:
@@
 Prog
 Text Notes 1750 6650 2    62   ~ 0
-VDD\nVPP\nVSS\nPGD\nPGC
+VPP\nVDD\nVSS\nPGD\nPGC
 Text GLabel 2000 4200 0    50   Input ~ 0
 PGD
